File: Circuit/AWG.kicad_pcb (KiCad board)
At the start: 2 copper layers, 47 x 45.7 mm, 24 parts, among them J1 Power, J2 Pump 1, J3 Pump 2, J4 Pump 3, J5 WL1, J6 Display, M1 Fan_3pin, M2 Fan_3pin, Q1 RFP30N06LE, Q2 RFP30N06LE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

Commit message: [Circuit] Update the footprints
Parts:
- J1: footprint Connector_PinHeader_2.54mm:PinHeader_1x04_P2.54mm_Vertical -> Connector_PinSocket_2.54mm:PinSocket_1x04_P2.54mm_Vertical
- moved M2 5.07 mm to (137.2, 77.5), turned to 0 degrees
- moved M1 5.06 mm to (128.3, 77.5), turned to 0 degrees
Connections:
- M1 pad 1: unconnected-(M1-Pad1) -> GND
- M1 pad 3: GND -> unconnected-(M1-Tacho-Pad3)
- M2 pad 1: unconnected-(M2-Pad1) -> GND
- M2 pad 3: GND -> unconnected-(M2-Tacho-Pad3)
