File: Circuit/AWG.kicad_sch (KiCad schematic)
At the start: 24 parts, among them J1 Power, J2 Pump 1, J3 Pump 2, J4 Pump 3, J5 WL1, J6 Display, M1 Fan_3pin, M2 Fan_3pin, Q1 RFP30N06LE, Q2 RFP30N06LE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

Commit message: [Circuit] Fix symbol warnings
Parts:
- J1, J6, PE1: symbol Connector:Conn_01x04_Male -> Connector:Conn_01x04_Pin
- J2, J3, J4: symbol Connector:Conn_01x02_Male -> Connector:Conn_01x02_Pin
- J5, U1: symbol Connector:Conn_01x03_Male -> Connector:Conn_01x03_Pin
- Q1, Q2: symbol Device:Q_NMOS_GDS -> Transistor_FET:Q_NMOS_GDS
- SW1: symbol Switch:SW_SPST_Lamp -> Switch:SW_SPST_LED
Connections:
- net GND: now also M1.1 (-), M2.1 (-); no longer M1.3 (-), M2.3 (-)

Commit message: [Circuit] Update the footprints
Parts:
- J1: footprint Connector_PinHeader_2.54mm:PinHeader_1x04_P2.54mm_Vertical -> Connector_PinSocket_2.54mm:PinSocket_1x04_P2.54mm_Vertical
Changed lines of the file:
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@@
 			)
 		)
-		(property "Footprint" "Connector_PinHeader_2.54mm:PinHeader_1x04_P2.54mm_Vertical"
+		(property "Footprint" "Connector_PinSocket_2.54mm:PinSocket_1x04_P2.54mm_Vertical"
 			(at 41.91 64.77 0)
 			(effects
